Commit message: 1

File: rover/urdf/gps.xacro (robot description, xacro)
@@ -19,5 +19,5 @@
 </link>
 <gazebo reference="gps_link">
-<material>Gazebo/Pink</material>
+<material>Gazebo/White</material>
 </gazebo>
 <joint name="gps_joint" type="fixed">

File: rover/urdf/rover.xacro (robot description, xacro)
@@ -1,8 +1,8 @@
 <?xml version='1.0'?>
-<robot name="atom" xmlns:xacro="http://www.ros.org/wiki/xacro">
-<xacro:include filename="$(find atom)/urdf/imu.xacro" />
-<xacro:include filename="$(find atom)/urdf/gps.xacro" />
-<xacro:include filename="$(find atom)/urdf/zed2.xacro" />
-	<xacro:property name="robot_name" value="atom" />
+<robot name="rover" xmlns:xacro="http://www.ros.org/wiki/xacro">
+<xacro:include filename="$(find rover)/urdf/imu.xacro" />
+<xacro:include filename="$(find rover)/urdf/gps.xacro" />
+<xacro:include filename="$(find rover)/urdf/zed2.xacro" />
+	<xacro:property name="robot_name" value="rover" />
 	<xacro:property name="robot_chassis_mass" value="15"/>
 	<xacro:property name="robot_chassis_length" value="0.2"/>
@@ -174,5 +174,5 @@
 			<origin xyz="0 0 0" rpy="0 0 0"/>
 			<geometry>
-				<mesh filename="package://atom/meshes/hokuyo.dae"/>
+				<mesh filename="package://rover/meshes/hokuyo.dae"/>
 			</geometry>
 		</visual>
@@ -286,4 +286,4 @@
 	</gazebo>
 	<!-- Motor, Camera and Lidar Simulation -->
-	<xacro:include filename="$(find atom)/urdf/atom.gazebo" />
+	<xacro:include filename="$(find rover)/urdf/rover.gazebo" />
 </robot>

File: rover/urdf/zed2.xacro (robot description, xacro)
@@ -25,5 +25,5 @@
 </link>
 <joint name="zed2_joint" type="fixed">
-    <origin xyz="0.26 0 0.05" rpy="0.0 1.57 1.57"/>
+    <origin xyz="0.26 0 0.05" rpy="0.0 0 0"/>
     <parent link="chassis"/>
     <child link="zed2_link"/>
@@ -33,10 +33,10 @@
 <link name="zed2_optical_frame"/>
 <joint name="zed2_optical_joint" type="fixed">
-  <origin xyz="0.0 0.0 0.0" rpy="1.57 -1.57 0.0"/>
+  <origin xyz="0.26 0 0.05" rpy="0 0 0.0"/>
   <parent link="zed2_link"/>
   <child link="zed2_optical_frame"/>
 </joint>
     <gazebo reference="zed2_optical_frame">
-    <material>Gazebo/Pink</material>
+    <material>Gazebo/Orange</material>
   <sensor name="zed2_optical_frame" type="depth">
     <update_rate>20</update_rate>
